Commit message: Use package:// URIs to make mesh discovery more robust

File: urdf/d435_camera.urdf.xacro (robot description, xacro)
@@ -10,5 +10,5 @@
                 <origin xyz="0 0 0" rpy="0 0 0" />
                 <geometry>
-                    <mesh filename="$(find walker_rosys)/meshes/realsense_d435.stl" />
+                    <mesh filename="package://walker_rosys/meshes/realsense_d435.stl" />
                 </geometry>
             </collision>
@@ -16,5 +16,5 @@
                 <origin xyz="0 0 0" rpy="1.57 0 1.57" />
                 <geometry>
-                    <mesh filename="$(find walker_rosys)/meshes/realsense_d435.stl" />
+                    <mesh filename="package://walker_rosys/meshes/realsense_d435.stl" />
                 </geometry>
             </visual>

File: urdf/walker.urdf (robot description, URDF)
Before this commit: robot walker_robot, 2 links, 1 joints
Links:
- link base_link: geometry collision mesh filename=package://walker_rosys/meshes/walker_frame.dae; visual mesh filename=package://walker_rosys/meshes/walker_frame.dae
